File: POVMEGA.brd (EAGLE design)
At the start: 85.1 x 57.7 mm, 12 parts

Commit message: sdfsd
sdf
Connections:
- net S$1 renamed S$18
Routing:
- net S$18: track 57.2 -> 84.3 mm
- net S$33: track 25.7 -> 0.00 mm
Changed lines of the file:
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@@
 <signal name="XT1R">
-</signal>
-<signal name="S$1">
-<wire x1="-27.305" y1="1.397" x2="10.795" y2="1.397" width="0.508" layer="1"/>
-<contactref element="E$9" pad="1"/>
-<wire x1="10.795" y1="1.397" x2="10.795" y2="-7.493" width="0.508" layer="1"/>
-<contactref element="E$3" pad="1"/>
-<wire x1="10.795" y1="-7.493" x2="14.605" y2="-7.493" width="0.508" layer="1"/>
-<wire x1="14.605" y1="-7.493" x2="14.605" y2="-13.843" width="0.508" layer="1"/>
 </signal>
 <signal name="S$2">
@@
 <wire x1="27.305" y1="19.304" x2="27.432" y2="19.177" width="0.508" layer="1"/>
 </signal>
-<signal name="S$33">
-<wire x1="-6.604" y1="-23.114" x2="-6.604" y2="-22.987" width="0.508" layer="1"/>
-<wire x1="-6.604" y1="-22.987" x2="-6.731" y2="-22.86" width="0.508" layer="1"/>
-<wire x1="-6.731" y1="-22.86" x2="-3.81" y2="-19.939" width="0.508" layer="1"/>
-<wire x1="-3.81" y1="-19.939" x2="-3.81" y2="1.143" width="0.508" layer="1"/>
-<wire x1="-3.81" y1="1.143" x2="-3.683" y2="1.27" width="0.508" layer="1"/>
-</signal>
 <signal name="S$35">
 <wire x1="-14.478" y1="-22.987" x2="-14.478" y2="-24.765" width="0.508" layer="16"/>
@@
 <wire x1="2.159" y1="14.097" x2="2.54" y2="14.478" width="0.508" layer="1"/>
 </signal>
+<signal name="S$18">
+<wire x1="-6.604" y1="-22.987" x2="-6.731" y2="-22.987" width="0.508" layer="1"/>
+<wire x1="-6.731" y1="-22.987" x2="-6.731" y2="-5.08" width="0.508" layer="1"/>
+<contactref element="E$9" pad="1"/>
+<wire x1="-27.305" y1="1.397" x2="-13.208" y2="1.397" width="0.508" layer="1"/>
+<wire x1="-13.208" y1="1.397" x2="10.795" y2="1.397" width="0.508" layer="1"/>
+<wire x1="10.795" y1="1.397" x2="10.795" y2="-7.493" width="0.508" layer="1"/>
+<contactref element="E$3" pad="1"/>
+<wire x1="10.795" y1="-7.493" x2="14.605" y2="-7.493" width="0.508" layer="1"/>
+<wire x1="14.605" y1="-7.493" x2="14.605" y2="-13.843" width="0.508" layer="1"/>
+<wire x1="-6.731" y1="-5.08" x2="-13.208" y2="1.397" width="0.508" layer="1"/>
+</signal>
 </signals>
